Commit message: 完成模型的更改 但插件和导航半径以及物理描述如质量等还未修改

File: panda_robot/panda_description/urdf/panda.urdf.xacro (robot description, xacro)
@@ -1,17 +1,18 @@
 <?xml version="1.0" ?>
 <!-- =================================================================================== -->
-<!-- |    This document was autogenerated by xacro from /opt/ros/kinetic/share/moveit_resources/panda_description/urdf/panda.urdf | -->
+<!-- |    This document was autogenerated by xacro from /opt/ros/kinetic/share/moveit_resourcespanda_description/urdf/panda.urdf | -->
 <!-- |    EDITING THIS FILE BY HAND IS NOT RECOMMENDED                                 | -->
 <!-- =================================================================================== -->
-<robot name="panda" xmlns:xacro="http://www.ros.org/wiki/xacro">
+<robot xmlns:xacro="http://www.ros.org/wiki/xacro">
+    <xacro:macro name= "arm_robot">
     <link name="panda_link0">
         <visual>
             <geometry>
-                <mesh filename="file://$(find moveit_resources_panda_description)/meshes/visual/link0.dae" />
-            </geometry>
-        </visual>
-        <collision>
-            <geometry>
-                <mesh filename="file://$(find moveit_resources_panda_description)/meshes/collision/link0.stl" />
+                <mesh filename="file://$(find panda_description)/meshes/visual/link0.dae" />
+            </geometry>
+        </visual>
+        <collision>
+            <geometry>
+                <mesh filename="file://$(find panda_description)/meshes/collision/link0.stl" />
             </geometry>
         </collision>
@@ -25,10 +26,10 @@
         <visual>
             <geometry>
-                <mesh filename="file://$(find moveit_resources_panda_description)/meshes/visual/link1.dae" />
-            </geometry>
-        </visual>
-        <collision>
-            <geometry>
-                <mesh filename="file://$(find moveit_resources_panda_description)/meshes/collision/link1.stl" />
+                <mesh filename="file://$(find panda_description)/meshes/visual/link1.dae" />
+            </geometry>
+        </visual>
+        <collision>
+            <geometry>
+                <mesh filename="file://$(find panda_description)/meshes/collision/link1.stl" />
             </geometry>
         </collision>
@@ -51,10 +52,10 @@
         <visual>
             <geometry>
-                <mesh filename="file://$(find moveit_resources_panda_description)/meshes/visual/link2.dae" />
-            </geometry>
-        </visual>
-        <collision>
-            <geometry>
-                <mesh filename="file://$(find moveit_resources_panda_description)/meshes/collision/link2.stl" />
+                <mesh filename="file://$(find panda_description)/meshes/visual/link2.dae" />
+            </geometry>
+        </visual>
+        <collision>
+            <geometry>
+                <mesh filename="file://$(find panda_description)/meshes/collision/link2.stl" />
             </geometry>
         </collision>
@@ -77,10 +78,10 @@
         <visual>
             <geometry>
-                <mesh filename="file://$(find moveit_resources_panda_description)/meshes/visual/link3.dae" />
-            </geometry>
-        </visual>
-        <collision>
-            <geometry>
-                <mesh filename="file://$(find moveit_resources_panda_description)/meshes/collision/link3.stl" />
+                <mesh filename="file://$(find panda_description)/meshes/visual/link3.dae" />
+            </geometry>
+        </visual>
+        <collision>
+            <geometry>
+                <mesh filename="file://$(find panda_description)/meshes/collision/link3.stl" />
             </geometry>
         </collision>
@@ -103,10 +104,10 @@
         <visual>
             <geometry>
-                <mesh filename="file://$(find moveit_resources_panda_description)/meshes/visual/link4.dae" />
-            </geometry>
-        </visual>
-        <collision>
-            <geometry>
-                <mesh filename="file://$(find moveit_resources_panda_description)/meshes/collision/link4.stl" />
+                <mesh filename="file://$(find panda_description)/meshes/visual/link4.dae" />
+            </geometry>
+        </visual>
+        <collision>
+            <geometry>
+                <mesh filename="file://$(find panda_description)/meshes/collision/link4.stl" />
             </geometry>
         </collision>
@@ -129,10 +130,10 @@
         <visual>
             <geometry>
-                <mesh filename="file://$(find moveit_resources_panda_description)/meshes/visual/link5.dae" />
-            </geometry>
-        </visual>
-        <collision>
-            <geometry>
-                <mesh filename="file://$(find moveit_resources_panda_description)/meshes/collision/link5.stl" />
+                <mesh filename="file://$(find panda_description)/meshes/visual/link5.dae" />
+            </geometry>
+        </visual>
+        <collision>
+            <geometry>
+                <mesh filename="file://$(find panda_description)/meshes/collision/link5.stl" />
             </geometry>
         </collision>
@@ -155,10 +156,10 @@
         <visual>
             <geometry>
-                <mesh filename="file://$(find moveit_resources_panda_description)/meshes/visual/link6.dae" />
-            </geometry>
-        </visual>
-        <collision>
-            <geometry>
-                <mesh filename="file://$(find moveit_resources_panda_description)/meshes/collision/link6.stl" />
+                <mesh filename="file://$(find panda_description)/meshes/visual/link6.dae" />
+            </geometry>
+        </visual>
+        <collision>
+            <geometry>
+                <mesh filename="file://$(find panda_description)/meshes/collision/link6.stl" />
             </geometry>
         </collision>
@@ -181,10 +182,10 @@
         <visual>
             <geometry>
-                <mesh filename="file://$(find moveit_resources_panda_description)/meshes/visual/link7.dae" />
-            </geometry>
-        </visual>
-        <collision>
-            <geometry>
-                <mesh filename="file://$(find moveit_resources_panda_description)/meshes/collision/link7.stl" />
+                <mesh filename="file://$(find panda_description)/meshes/visual/link7.dae" />
+            </geometry>
+        </visual>
+        <collision>
+            <geometry>
+                <mesh filename="file://$(find panda_description)/meshes/collision/link7.stl" />
             </geometry>
         </collision>
@@ -219,10 +220,10 @@
         <visual>
             <geometry>
-                <mesh filename="file://$(find moveit_resources_panda_description)/meshes/visual/hand.dae" />
-            </geometry>
-        </visual>
-        <collision>
-            <geometry>
-                <mesh filename="file://$(find moveit_resources_panda_description)/meshes/collision/hand.stl" />
+                <mesh filename="file://$(find panda_description)/meshes/visual/hand.dae" />
+            </geometry>
+        </visual>
+        <collision>
+            <geometry>
+                <mesh filename="file://$(find panda_description)/meshes/collision/hand.stl" />
             </geometry>
         </collision>
@@ -236,10 +237,10 @@
         <visual>
             <geometry>
-                <mesh filename="file://$(find moveit_resources_panda_description)/meshes/visual/finger.dae" />
-            </geometry>
-        </visual>
-        <collision>
-            <geometry>
-                <mesh filename="file://$(find moveit_resources_panda_description)/meshes/collision/finger.stl" />
+                <mesh filename="file://$(find panda_description)/meshes/visual/finger.dae" />
+            </geometry>
+        </visual>
+        <collision>
+            <geometry>
+                <mesh filename="file://$(find panda_description)/meshes/collision/finger.stl" />
             </geometry>
         </collision>
@@ -254,5 +255,5 @@
             <origin rpy="0 0 3.14159265359" xyz="0 0 0" />
             <geometry>
-                <mesh filename="file://$(find moveit_resources_panda_description)/meshes/visual/finger.dae" />
+                <mesh filename="file://$(find panda_description)/meshes/visual/finger.dae" />
             </geometry>
         </visual>
@@ -260,5 +261,5 @@
             <origin rpy="0 0 3.14159265359" xyz="0 0 0" />
             <geometry>
-                <mesh filename="file://$(find moveit_resources_panda_description)/meshes/collision/finger.stl" />
+                <mesh filename="file://$(find panda_description)/meshes/collision/finger.stl" />
             </geometry>
         </collision>
@@ -286,3 +287,4 @@
         <dynamics damping="0.3" />
     </joint>
+    </xacro:macro>
 </robot>

File: robot/urdf/project_robot/plugins/gazebo_sensor_plugin.xacro (robot description, xacro)
@@ -34,7 +34,8 @@
                 </scan>
                 <!-- 设置扫描距离 -->
+                <!-- 修改 -->
                 <range>
-                    <min>0.120000</min>
-                    <max>8.0</max>
+                    <min>0.250000</min>
+                    <max>12.0</max>
                     <resolution>0.015000</resolution>
                 </range>

File: robot/urdf/project_robot/robot.urdf.xacro (robot description, xacro)
@@ -17,16 +17,25 @@
     <xacro:include filename='$(find robot)/urdf/project_robot/plugins/gazebo_sensor_plugin.xacro'/>
     <xacro:include filename='$(find robot)/urdf/project_robot/ros2_control.xacro'/>
+    <!-- panda arm robot -->
+    <xacro:include filename='$(find panda_description)/urdf/panda.urdf.xacro'/>
     <!-- 使用宏 -->
     <!-- 使用宏传入坐标时要使轮子在一个地面 调试中修改 -->
-    <xacro:base_xacro length='0.12' radius='0.10'/>
+    <xacro:base_xacro length='0.16' radius='0.22'/>
     <xacro:imu_xacro xyz='0.0 0.0 0.02'/>
-    <xacro:camera_xacro xyz='0.10 0.0 0.075'/>
-    <xacro:laser_xacro xyz='0.0 0.0 0.11'/>
-    <xacro:wheel_xacro wheel_name='left_wheel' xyz='0 0.10 -0.06'/>
-    <xacro:wheel_xacro wheel_name='right_wheel' xyz='0 -0.10 -0.06'/>
-    <xacro:caster_xacro caster_name='front_caster' xyz='0.08 0 -0.076'/>
-    <xacro:caster_xacro caster_name='back_caster' xyz='-0.08 0 -0.076'/>
+    <xacro:camera_xacro xyz='0.23 0.0 0.075'/>
+    <xacro:laser_xacro xyz='0.17 0.0 0.12'/>
+    <xacro:wheel_xacro wheel_name='left_wheel' xyz='0 0.25 -0.08'/>
+    <xacro:wheel_xacro wheel_name='right_wheel' xyz='0 -0.25 -0.08'/>
+    <xacro:caster_xacro caster_name='front_caster' xyz='0.2 0 -0.096'/>
+    <xacro:caster_xacro caster_name='back_caster' xyz='-0.2 0 -0.096'/>
     <!-- <xacro:gazebo_control_plugin/> -->
     <xacro:gazebo_sensor_plugin/>
     <xacro:ros2_control/>
+    <!--机械臂 -->
+    <!-- <xacro:arm_robot/>
+    <joint name="chassis_to_arm_joint" type="fixed">
+        <parent link="base_link"/>
+        <child link="panda_link0"/>
+        <origin xyz="0.0 0.0 0.06" rpy="0.0 0.0 0.0"/>
+    </joint> -->
 </robot>

File: robot/urdf/project_robot/sensor/imu.urdf.xacro (robot description, xacro)
@@ -9,5 +9,5 @@
                 <origin xyz="0.0 0.0 0.0" rpy="0.0 0.0 0.0"/>
                 <geometry>
-                    <box size="0.02 0.02 0.02"/>
+                    <box size="0.04 0.04 0.04"/>
                 </geometry>
                 <material name = 'black'>
@@ -18,5 +18,5 @@
                 <origin xyz="0.0 0.0 0.0" rpy="0.0 0.0 0.0"/>
                 <geometry>
-                    <box size="0.02 0.02 0.02"/>
+                    <box size="0.04 0.04 0.04"/>
                 </geometry>
                 <material name = 'black'>

File: robot/urdf/project_robot/sensor/laser.urdf.xacro (robot description, xacro)
@@ -10,5 +10,5 @@
                 <origin xyz="0.0 0.0 0.0" rpy="0.0 0.0 0.0"/>
                 <geometry>
-                        <cylinder radius="0.01" length="0.10"/>
+                        <cylinder radius="0.01" length="0.06"/>
                 </geometry>
                 <material name = 'black'>
@@ -19,5 +19,5 @@
                 <origin xyz="0.0 0.0 0.0" rpy="0.0 0.0 0.0"/>
                 <geometry>
-                        <cylinder radius="0.01" length="0.10"/>
+                        <cylinder radius="0.01" length="0.06"/>
                 </geometry>
                 <material name = 'black'>
@@ -54,5 +54,5 @@
         <joint name="laser_joint" type="fixed">
             <!-- 计算雷达杆几何中心 将雷达固定到雷达杆上 -->
-            <origin xyz="0.0 0.0 0.05" rpy="0.0 0.0 0.0"/>
+            <origin xyz="0.0 0.0 0.03" rpy="0.0 0.0 0.0"/>
             <parent link="laser_cylinder_link"/>
             <child link="laser_link"/>
